File: DPS/Bluetooth.brd (EAGLE design)
At the start: 17 parts

Commit message: Summar dps
Parts:
- removed E$11: (no value), capacitor-wima:C2.5-2
- removed E$12, E$15, E$20: (no value), led:LED3MM
- removed E$14, E$9: (no value), eagle-ltspice:0204/7
- removed E$3: (no value), crystal:HC49/S
- E$10: device eagle-ltspice:0204/7 -> con-lstb:MA03-1
- moved E$10 5.53 mm to (75.4, 54.9), turned to 180 degrees
Routing:
- net S$37: track 16.3 -> 0.00 mm
- net S$36: track 15.7 -> 0.00 mm
- net S$35: track 14.0 -> 0.00 mm
- net S$27: track 0.00 -> 8.00 mm
- net S$33: track 7.82 -> 0.00 mm
- net S$28: track 3.26 -> 8.12 mm
- net S$29: track 5.16 -> 8.06 mm
Other:
- board text added: "Bluetooth"
- board text added: "Layer 1"
- board text removed: "Master"
Changed lines of the file:
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@@
 <plain>
 <text x="93.4" y="44.21" size="2.1844" layer="16" rot="MR0">DOMINIK TKACIK</text>
-<text x="35.52" y="80.69" size="3.81" layer="16" rot="MR180">Master </text>
 <rectangle x1="84.155" y1="78.845" x2="87.165" y2="80.165" layer="16" rot="R90"/>
 <rectangle x1="82.155" y1="78.845" x2="85.165" y2="80.165" layer="16" rot="R90"/>
@@
 <text x="33.44" y="52.17" size="1.27" layer="16" rot="MR0">3V3</text>
 <text x="62.08" y="82.67" size="2.54" layer="16" rot="MR180">868 MHZ</text>
+<text x="51" y="78" size="2.54" layer="16" rot="MR0">Bluetooth</text>
+<text x="94" y="56" size="2.54" layer="16" rot="MR0">Layer 1</text>
 </plain>
 <attributes>
@@
 <element name="E$5" library="resistor" package="0207/10" value="" x="36.85" y="58.09"/>
 <element name="E$6" library="switch" package="TL1105T" value="" x="36.83" y="64.77"/>
-<element name="E$9" library="eagle-ltspice" package="0204/7" value="" x="77.57" y="55.86" rot="R180"/>
-<element name="E$10" library="eagle-ltspice" package="0204/7" value="" x="80.08" y="57.84"/>
-<element name="E$12" library="led" package="LED3MM" value="" x="96.52" y="56.87"/>
 <element name="E$7" library="transistor-pnp" package="TO220" value="" x="43.25" y="52.24" rot="R270"/>
 <element name="E$19" library="capacitor-wima" package="C2.5-2" value="" x="63.48" y="51.78" rot="R90"/>
 <element name="E$8" library="con-lstb" package="MA04-1" value="" x="49.58" y="54.92"/>
 <element name="E$13" library="pinhead" package="1X02" value="" x="32.41" y="50.89" rot="R90"/>
-<element name="E$14" library="eagle-ltspice" package="0204/7" value="" x="75.57" y="53.86" rot="R180"/>
-<element name="E$15" library="led" package="LED3MM" value="" x="96.63" y="53.09"/>
-<element name="E$20" library="led" package="LED3MM" value="" x="96.47" y="60.64"/>
 <element name="E$2" library="capacitor-wima" package="C2.5-2" value="" x="66.19" y="51.79" rot="R90"/>
-<element name="E$3" library="crystal" package="HC49/S" value="" x="64.77" y="57.15"/>
-<element name="E$11" library="capacitor-wima" package="C2.5-2" value="" x="66.19" y="51.79" rot="R90"/>
 <element name="E$1" library="atmega328L" package="DIL28-3" value="" x="59.75" y="65.13"/>
+<element name="E$10" library="con-lstb" package="MA03-1" value="" x="75.39" y="54.91" rot="R180"/>
 </elements>
 <signals>
@@
 <via x="34.57" y="68.02" extent="1-16" drill="0.5" diameter="3"/>
 <via x="39.09" y="68" extent="1-16" drill="0.5" diameter="3"/>
-<wire x1="34.57" y1="68.02" x2="39.09" y2="68" width="0" layer="19" extent="1-1"/>
 <via x="41.97" y="57.84" extent="1-16" drill="0.5" diameter="3"/>
 <via x="39.1" y="61.49" extent="1-16" drill="0.5" diameter="3"/>
-<wire x1="39.1" y1="61.49" x2="41.97" y2="57.84" width="0" layer="19" extent="1-1"/>
-<wire x1="39.09" y1="68" x2="39.1" y2="61.49" width="0" layer="19" extent="1-1"/>
 <via x="34.55" y="61.5" extent="1-16" drill="0.5" diameter="3"/>
+<via x="31.85" y="58.05" extent="1-16" drill="0.5" diameter="3"/>
+<via x="80.06" y="79.47" extent="1-16" drill="0.5" diameter="3"/>
+<wire x1="39.09" y1="68" x2="80.06" y2="79.47" width="0" layer="19" extent="1-1"/>
+<wire x1="34.57" y1="68.02" x2="39.09" y2="68" width="0" layer="19" extent="1-1"/>
+<wire x1="39.1" y1="61.49" x2="39.09" y2="68" width="0" layer="19" extent="1-1"/>
 <wire x1="34.55" y1="61.5" x2="39.1" y2="61.49" width="0" layer="19" extent="1-1"/>
-<via x="31.85" y="58.05" extent="1-16" drill="0.5" diameter="3"/>
 <wire x1="31.85" y1="58.05" x2="34.55" y2="61.5" width="0" layer="19" extent="1-1"/>
-<via x="80.06" y="79.47" extent="1-16" drill="0.5" diameter="3"/>
+<wire x1="41.97" y1="57.84" x2="39.1" y2="61.49" width="0" layer="19" extent="1-1"/>
 </signal>
 <signal name="S$30">
@@
 <via x="63.4" y="49.85" extent="1-16" drill="0.5" diameter="3"/>
 <via x="66.73" y="49.84" extent="1-16" drill="0.5" diameter="3"/>
-<via x="98.17" y="60.59" extent="1-16" drill="0.5" diameter="3"/>
-<via x="98.18" y="56.8" extent="1-16" drill="0.5" diameter="3"/>
-<via x="98.37" y="53.06" extent="1-16" drill="0.5" diameter="3"/>
-<via x="95.12" y="53.05" extent="1-16" drill="0.5" diameter="3"/>
-<via x="95.1" y="56.84" extent="1-16" drill="0.5" diameter="3"/>
-<via x="95.09" y="60.65" extent="1-16" drill="0.5" diameter="3"/>
-<via x="83.98" y="57.88" extent="1-16" drill="0.5" diameter="3"/>
-<via x="81.41" y="55.8" extent="1-16" drill="0.5" diameter="3"/>
-<via x="79.18" y="53.63" extent="1-16" drill="0.5" diameter="3"/>
-<via x="71.66" y="53.82" extent="1-16" drill="0.5" diameter="2.5"/>
-<via x="73.94" y="56" extent="1-16" drill="0.5" diameter="2.5"/>
-<via x="76.37" y="57.92" extent="1-16" drill="0.5" diameter="2.5"/>
 <via x="55.89" y="47.34" extent="1-16" drill="0.5" diameter="3"/>
-<wire x1="95.09" y1="60.65" x2="98.17" y2="60.59" width="0" layer="19" extent="1-1"/>
-<wire x1="98.18" y1="56.8" x2="98.17" y2="60.59" width="0" layer="19" extent="1-1"/>
-<wire x1="95.1" y1="56.84" x2="98.18" y2="56.8" width="0" layer="19" extent="1-1"/>
-<wire x1="98.37" y1="53.06" x2="98.18" y2="56.8" width="0" layer="19" extent="1-1"/>
-<wire x1="95.12" y1="53.05" x2="98.37" y2="53.06" width="0" layer="19" extent="1-1"/>
-<wire x1="83.98" y1="57.88" x2="95.1" y2="56.84" width="0" layer="19" extent="1-1"/>
-<wire x1="81.41" y1="55.8" x2="83.98" y2="57.88" width="0" layer="19" extent="1-1"/>
-<wire x1="79.18" y1="53.63" x2="81.41" y2="55.8" width="0" layer="19" extent="1-1"/>
-<wire x1="76.37" y1="57.92" x2="79.18" y2="53.63" width="0" layer="19" extent="1-1"/>
-<wire x1="73.94" y1="56" x2="76.37" y2="57.92" width="0" layer="19" extent="1-1"/>
-<wire x1="71.66" y1="53.82" x2="73.94" y2="56" width="0" layer="19" extent="1-1"/>
-<wire x1="66.71" y1="53.13" x2="71.66" y2="53.82" width="0" layer="19" extent="1-1"/>
+<via x="60.81" y="47.27" extent="1-16" drill="0.5" diameter="3"/>
 <wire x1="66.73" y1="49.84" x2="66.71" y2="53.13" width="0" layer="19" extent="1-1"/>
 <wire x1="63.37" y1="53.09" x2="66.71" y2="53.13" width="0" layer="19" extent="1-1"/>
 <wire x1="63.4" y1="49.85" x2="63.37" y2="53.09" width="0" layer="19" extent="1-1"/>
+<wire x1="60.81" y1="47.27" x2="63.4" y2="49.85" width="0" layer="19" extent="1-1"/>
 <wire x1="62.71" y1="57.13" x2="63.37" y2="53.09" width="0" layer="19" extent="1-1"/>
 <wire x1="67.71" y1="57.13" x2="66.71" y2="53.13" width="0" layer="19" extent="1-1"/>
-<wire x1="55.89" y1="47.34" x2="63.4" y2="49.85" width="0" layer="19" extent="1-1"/>
-<wire x1="55.82" y1="47.35" x2="55.89" y2="47.34" width="0" layer="19" extent="1-1"/>
-<via x="60.81" y="47.27" extent="1-16" drill="0.5" diameter="3"/>
-</signal>
-<signal name="S$45">
-<wire x1="63.47" y1="53.41" x2="66.05" y2="53.46" width="0" layer="19" extent="1-1"/>
+<wire x1="55.89" y1="47.34" x2="60.81" y2="47.27" width="0" layer="19" extent="1-1"/>
 </signal>
 <signal name="S$16">
@@
 <wire x1="85.68" y1="76.4" x2="85.66" y2="78.65" width="1.6764" layer="16"/>
 </signal>
-<signal name="S$28">
-<wire x1="76.28" y1="61.12" x2="76.28" y2="57.86" width="1.6764" layer="16"/>
-</signal>
-<signal name="S$29">
-<wire x1="73.63" y1="61.12" x2="73.63" y2="55.96" width="1.6764" layer="16"/>
-</signal>
-<signal name="S$33">
-<wire x1="71.22" y1="61.23" x2="71.22" y2="53.99" width="1.6764" layer="16"/>
-<wire x1="71.22" y1="53.99" x2="71.8" y2="53.99" width="1.6764" layer="16"/>
-</signal>
-<signal name="S$35">
-<wire x1="84.05" y1="57.83" x2="84.05" y2="60.68" width="1.6764" layer="16"/>
-<wire x1="84.05" y1="60.68" x2="95.19" y2="60.68" width="1.6764" layer="16"/>
-</signal>
-<signal name="S$36">
-<wire x1="81.5" y1="55.36" x2="86.63" y2="55.36" width="1.6764" layer="16"/>
-<wire x1="86.63" y1="55.36" x2="86.6" y2="56.98" width="1.6764" layer="16"/>
-<wire x1="86.6" y1="56.98" x2="95.56" y2="56.98" width="1.6764" layer="16"/>
-</signal>
-<signal name="S$37">
-<wire x1="79.37" y1="53.11" x2="95.63" y2="53.11" width="1.6764" layer="16"/>
-</signal>
 <signal name="S$1">
 <wire x1="63.45" y1="60.93" x2="63.45" y2="52.99" width="1.6764" layer="16"/>
@@
 <wire x1="29.12" y1="52.21" x2="29.12" y2="52.31" width="1.6764" layer="16"/>
 </signal>
+<signal name="S$27">
+<wire x1="76.26" y1="61.24" x2="77.95" y2="61.24" width="1.6764" layer="16"/>
+<wire x1="77.95" y1="61.24" x2="77.95" y2="54.93" width="1.6764" layer="16"/>
+</signal>
+<signal name="S$28">
+<wire x1="73.73" y1="61.24" x2="73.73" y2="58.25" width="1.6764" layer="16"/>
+<wire x1="73.73" y1="58.25" x2="75.38" y2="58.25" width="1.6764" layer="16"/>
+<wire x1="75.38" y1="58.25" x2="75.38" y2="54.77" width="1.6764" layer="16"/>
+</signal>
+<signal name="S$29">
+<wire x1="71.19" y1="61.27" x2="71.19" y2="54.87" width="1.6764" layer="16"/>
+<wire x1="71.19" y1="54.87" x2="72.85" y2="54.87" width="1.6764" layer="16"/>
+</signal>
 </signals>
