File: DPS/Bluetooth2layer.brd (EAGLE design)
At the start: 17 parts

Commit message: Summar dps
Parts:
- removed E$11, E$19: (no value), capacitor-wima:C2.5-2
- removed E$12, E$15, E$20: (no value), led:LED3MM
- removed E$13: (no value), pinhead:1X02
- removed E$14, E$9: (no value), eagle-ltspice:0204/7
- E$1: device atmega328L:DIL28-3 -> rcl:0207/10
- E$10: device eagle-ltspice:0204/7 -> con-lstb:MA03-1
- E$2: device capacitor-wima:C2.5-2 -> rcl:0207/10
- E$3: device crystal:HC49/S -> rcl:0207/10
- E$4: device crystal:HC49/S -> led:LED3MM
- E$5: device resistor:0207/10 -> led:LED3MM
- E$6: device switch:TL1105T -> led:LED3MM
- E$7: device transistor-pnp:TO220 -> con-lstb:MA04-1
- moved E$5 26.2 mm to (63.0, 56.0), turned to 270 degrees
- moved E$6 22.9 mm to (58.0, 56.0), turned to 270 degrees
- moved E$1 18.3 mm to (78.0, 64.0), turned to 90 degrees
- moved E$2 17.4 mm to (75.4, 66.5)
- moved E$7 13.6 mm to (46.1, 65.6), turned to 90 degrees
- moved E$3 10.5 mm to (72.8, 64.0), turned to 90 degrees
- moved E$10 5.53 mm to (75.4, 54.9), turned to 180 degrees
- moved E$4 3.43 mm to (68.0, 56.0), turned to 270 degrees
Routing:
- net S$22: track 84.0 -> 0.00 mm
- net S$32: track 63.8 -> 0.00 mm
- net S$44: track 60.0 -> 0.00 mm
- net S$38: track 58.0 -> 0.00 mm
- net S$17: track 50.1 -> 0.00 mm
- net S$3: track 48.3 -> 4.04 mm
- net S$18: track 36.3 -> 0.00 mm
- net S$19: track 31.8 -> 0.00 mm
- net S$21: track 30.2 -> 0.00 mm
- net S$24: track 29.5 -> 0.00 mm
- net S$7: track 9.63 -> 26.7 mm
- net S$37: track 16.3 -> 0.00 mm
- net S$36: track 15.7 -> 0.00 mm
- net S$6: track 37.3 -> 22.0 mm
- net S$35: track 14.0 -> 0.00 mm
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Other:
- board text added: "Bluetooth"
- board text added: "Layer2"
- board text removed: "3V3"
- board text removed: "3V3 - 16V"
- board text removed: "868 MHZ"
- board text removed: "DOMINIK TKACIK"
- board text removed: "GND"
- board text removed: "Master"
