File: DPS/codeLock.brd (EAGLE design)
At the start: 17 parts

Commit message: Summar dps
Parts:
- removed E$10, E$14, E$9: (no value), eagle-ltspice:0204/7
- removed E$12, E$15, E$20: (no value), led:LED3MM
- removed E$3: (no value), crystal:HC49/S
- added E$16: (no value), con-lstb:MA06-1
- E$2: device capacitor-wima:C2.5-2 -> con-lstb:MA05-1
- moved E$2 9.58 mm to (73.7, 57.8), turned to 0 degrees
- moved E$19 7.12 mm to (68.2, 46.4)
- moved E$4 5.59 mm to (66.2, 51.8)
- moved E$11 5.59 mm to (64.5, 46.5)
Routing:
- net S$22: track 84.0 -> 53.0 mm
- net S$37: track 16.3 -> 0.00 mm
- net S$36: track 15.7 -> 0.00 mm, vias 0 -> 1
- net S$31: track 1.18 -> 16.5 mm
- net S$38: track 58.0 -> 70.0 mm
- net S$35: track 14.0 -> 3.38 mm
- net S$11: track 10.2 -> 18.2 mm
- net S$1: track 7.98 -> 0.00 mm, vias 0 -> 1
- net S$42: track 0.00 -> 6.25 mm
- net S$34: track 0.00 -> 6.24 mm
- net S$41: track 0.00 -> 6.19 mm
- net S$27: track 0.00 -> 6.19 mm
- net S$40: track 0.00 -> 6.18 mm
- net S$32: track 63.8 -> 69.4 mm
- net S$29: track 5.16 -> 0.00 mm, vias 0 -> 1
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Other:
- board text added: "Code Lock"
- board text removed: "Master"
