File: DPS/codeLock2layer.brd (EAGLE design)
At the start: 17 parts

Commit message: Summar dps
Parts:
- removed E$10, E$14, E$9: (no value), eagle-ltspice:0204/7
- removed E$11, E$19: (no value), capacitor-wima:C2.5-2
- removed E$12, E$15, E$20: (no value), led:LED3MM
- removed E$13: (no value), pinhead:1X02
- removed E$7: (no value), transistor-pnp:TO220
- removed E$8: (no value), con-lstb:MA04-1
- added E$16: (no value), con-lstb:MA06-1
- E$1: device atmega328L:DIL28-3 -> con-lstb:MA08-1
- E$2: device capacitor-wima:C2.5-2 -> con-lstb:MA05-1
- E$3, E$4: device crystal:HC49/S -> rcl:0207/10
- E$5: device resistor:0207/10 -> led:LED3MM
- E$6: device switch:TL1105T -> led:LED3MM
- moved E$5 44.5 mm to (78.0, 75.0), turned to 180 degrees
- moved E$6 41.6 mm to (78.0, 71.0), turned to 180 degrees
- moved E$4 13.6 mm to (69.3, 70.0), turned to 90 degrees
- moved E$3 12.9 mm to (65.4, 70.1), turned to 90 degrees
- moved E$2 9.58 mm to (73.7, 57.8), turned to 0 degrees
- moved E$1 9.50 mm to (52.2, 70.9)
Routing:
- net S$22: track 84.0 -> 0.00 mm
- net S$32: track 63.8 -> 0.00 mm
- net S$44: track 60.0 -> 0.00 mm
- net S$38: track 58.0 -> 0.00 mm
- net S$17: track 50.1 -> 0.00 mm
- net S$6: track 37.3 -> 0.00 mm, vias 0 -> 8
- net S$18: track 36.3 -> 0.00 mm
- net S$12: track 32.8 -> 0.00 mm
- net S$19: track 31.8 -> 0.00 mm
- net S$21: track 30.2 -> 0.00 mm
- net S$24: track 29.5 -> 0.00 mm
- net S$3: track 48.3 -> 24.4 mm
- net S$37: track 16.3 -> 0.00 mm
- net S$36: track 15.7 -> 0.00 mm
- net S$1: track 7.98 -> 23.1 mm
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Other:
- board text added: "CodeLock Layer 2"
- board text removed: "3V3"
- board text removed: "3V3 - 16V"
- board text removed: "868 MHZ"
- board text removed: "DOMINIK TKACIK"
- board text removed: "GND"
- board text removed: "Master"
