File: gate-modules/Dps/Gate.brd (EAGLE design)
At the start: 17 parts

Commit message: >)
Parts:
- removed E$14: (no value), eagle-ltspice:0204/7
- removed E$20: (no value), led:LED3MM
- added E$16: (no value), rcl:C050-030X075
- added E$17, E$18: (no value), relay:CQ1
- E$10, E$9: device eagle-ltspice:0204/7 -> diode:C5102
- E$12: device led:LED3MM -> con-wago-500:W237-136
- E$15: device led:LED3MM -> special:EDG-04
- moved E$15 50.0 mm to (52.1, 75.9)
- moved E$12 44.6 mm to (56.2, 37.7)
- moved E$9 15.4 mm to (92.9, 56.2), turned to 0 degrees
- moved E$10 2.31 mm to (78.4, 56.2), turned to 180 degrees
- moved E$7 2.00 mm to (45.2, 52.2)
Routing:
- net S$57: track 0.00 -> 73.7 mm
- net S$22: track 84.0 -> 11.1 mm
- net S$56: track 0.00 -> 72.7 mm
- net S$53: track 0.00 -> 46.5 mm
- net S$32: track 63.8 -> 105.3 mm
- net S$27: track 0.00 -> 35.6 mm
- net S$17: track 50.1 -> 17.7 mm
- net S$52: track 0.00 -> 30.0 mm
- net S$11: track 10.2 -> 39.9 mm
- net S$49: track 0.00 -> 28.4 mm
- net S$12: track 32.8 -> 6.69 mm
- net S$47: track 0.00 -> 24.4 mm
- net S$50: track 0.00 -> 18.9 mm
- net S$58: track 0.00 -> 14.0 mm
- net S$28: track 3.26 -> 17.0 mm
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Other:
- board text added: "Gate"
- board text removed: "3V3"
- board text removed: "Master"
