File: masters/arduinoMaster/master/dps/Master.brd (EAGLE design)
At the start: 10 parts

Commit message: >)
Parts:
- added E$11: (no value), capacitor-wima:C2.5-2
- added E$12, E$15, E$20: (no value), led:LED3MM
- added E$14, E$9: (no value), eagle-ltspice:0204/7
- added E$16: (no value), rcl:C050-030X075
- added E$3: (no value), crystal:HC49/S
- E$10: device con-lstb:MA03-1 -> eagle-ltspice:0204/7
- moved E$10 5.53 mm to (80.1, 57.8), turned to 0 degrees
- moved E$7 1.35 mm to (44.6, 52.2)
Routing:
- net S$17: track 50.1 -> 17.7 mm
- net S$27: track 8.00 -> 35.6 mm
- net S$37: track 0.00 -> 16.3 mm
- net S$36: track 0.00 -> 15.7 mm
- net S$35: track 0.00 -> 14.0 mm
- net S$43: track 0.00 -> 11.5 mm
- net S$11: track 10.2 -> 0.00 mm
- net S$33: track 0.00 -> 7.82 mm
- net S$44: track 60.0 -> 67.0 mm
- net S$38: track 58.0 -> 64.0 mm
- net S$42: track 0.00 -> 4.90 mm
- net S$28: track 8.12 -> 3.26 mm
- net S$10: track 4.70 -> 8.64 mm
- net S$9: track 4.99 -> 7.93 mm
- net S$29: track 8.06 -> 5.16 mm
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Other:
- board text added: "Master"
- board text removed: "3V3"
- board text removed: "Bluetooth"
- board text removed: "Layer 1"
