File: opening-modules/cardreader/DPS/readCard.brd (EAGLE design)
At the start: 11 parts

Commit message: >)
Parts:
- removed E$16: (no value), con-lstb:MA06-1
- removed E$2: (no value), con-lstb:MA05-1
- added E$3: (no value), rcl:C050-025X075
- added E$9: (no value), con-lstb:MA07-1
- moved E$7 1.52 mm to (44.8, 52.3)
Routing:
- net S$40: track 6.18 -> 48.1 mm
- net S$49: track 0.00 -> 41.3 mm
- net S$37: track 0.00 -> 33.3 mm
- net S$17: track 50.1 -> 21.1 mm
- net S$27: track 6.19 -> 25.4 mm
- net S$3: track 48.3 -> 66.3 mm
- net S$32: track 69.4 -> 82.7 mm
- net S$33: track 12.7 -> 23.6 mm
- net S$46: track 0.00 -> 9.60 mm
- net S$11: track 18.2 -> 25.3 mm
- net S$38: track 70.0 -> 63.4 mm
- net S$42: track 6.25 -> 0.00 mm, vias 0 -> 1
- net S$34: track 6.24 -> 0.00 mm
- net S$41: track 6.19 -> 0.00 mm, vias 0 -> 1
- net S$31: track 16.5 -> 11.7 mm
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Other:
- board text removed: "3V3"
- board text removed: "Code Lock"
