File: opening-modules/code-lock/DPS/codeLock.brd (EAGLE design)
At the start: 11 parts

Commit message: >)
Parts:
- removed E$16: (no value), con-lstb:MA06-1
- added E$12, E$9: (no value), con-lstb:MA05-1
- added E$3: (no value), rcl:C050-025X075
- E$2: device con-lstb:MA05-1 -> buzzer:F/QMBIII
- moved E$2 17.8 mm to (90.6, 52.4), turned to 180 degrees
- moved E$7 1.52 mm to (44.8, 52.3)
Connections:
- new net S$49: E$1.11
Routing:
- net S$25: track 6.08 -> 48.2 mm
- net S$37: track 0.00 -> 33.3 mm
- net S$17: track 50.1 -> 21.1 mm
- net S$46: track 0.00 -> 12.6 mm
- net S$53: track 0.00 -> 5.55 mm
- net S$31: track 16.5 -> 11.7 mm
- net S$52: track 0.00 -> 4.66 mm
- net S$49: track 0.00 -> 4.63 mm
- net S$51: track 0.00 -> 4.60 mm
- net S$50: track 0.00 -> 4.57 mm
- net S$48: track 0.00 -> 4.43 mm
- net S$18: track 36.3 -> 32.3 mm
- net S$9: track 4.99 -> 8.93 mm
- net S$10: track 4.70 -> 8.64 mm
- net S$32: track 69.4 -> 72.7 mm
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Other:
- board text added: "CodeLock"
- board text removed: "3V3"
- board text removed: "Code Lock"
